File: DIFF_BOARD_REV2.kicad_sch (KiCad schematic)
At the start: 0 parts

Commit message: updated silkscreen
Other:
- title: TeensyDAQ -> DIFF BOARD REV2
Changed lines of the file:
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@@
 	(paper "A4")
 	(title_block
-		(title "TeensyDAQ")
+		(title "DIFF BOARD REV2")
 		(date "2025-02-11")
 		(rev "0")
